Commit message: Change shape of spoon handle. Add world_idx feature. Fix world_random_scale feature.

File: robo_manip_baselines/envs/assets/tacto/objects/spoon/dummy_spoon.urdf (robot description, URDF)
Before this commit: robot dummy_spoon.urdf, 1 links, 0 joints
Links:
- link spoon: mass 0.01 -> 0.02; geometry collision box size=0.08 0.16 0.7; collision sphere radius=0.17
