Commit message: Add and use spoon mesh. Adjust boxes and spoon. Add ReachPhase as pre-motion phase.

File: robo_manip_baselines/envs/assets/tacto/objects/box/blue_box.urdf (robot description, URDF)
Before this commit: robot blue_box.urdf, 5 links, 4 joints
Links:
- link bottom: geometry collision box size=0.3 0.3 0.1; visual box size=0.3 0.3 0.1
- link edge_nx: geometry collision box size=0.025 0.3 0.5; visual box size=0.025 0.3 0.5
- link edge_ny: geometry collision box size=0.3 0.025 0.5; visual box size=0.3 0.025 0.5
- link edge_px: geometry collision box size=0.025 0.3 0.5; visual box size=0.025 0.3 0.5
- link edge_py: geometry collision box size=0.3 0.025 0.5; visual box size=0.3 0.025 0.5
Joints:
- joint edge_joint_nx: origin xyz=-0.225 0 0 -> xyz=-0.1455 0 0
- joint edge_joint_ny: origin xyz=0 -0.225 0 -> xyz=0 -0.1455 0
- joint edge_joint_px: origin xyz=0.225 0 0 -> xyz=0.1455 0 0
- joint edge_joint_py: origin xyz=0 0.225 0 -> xyz=0 0.1455 0

File: robo_manip_baselines/envs/assets/tacto/objects/box/green_box.urdf (robot description, URDF)
Before this commit: robot green_box.urdf, 5 links, 4 joints
Links:
- link bottom: geometry collision box size=0.3 0.3 0.1; visual box size=0.3 0.3 0.1
- link edge_nx: geometry collision box size=0.025 0.3 0.5; visual box size=0.025 0.3 0.5
- link edge_ny: geometry collision box size=0.3 0.025 0.5; visual box size=0.3 0.025 0.5
- link edge_px: geometry collision box size=0.025 0.3 0.5; visual box size=0.025 0.3 0.5
- link edge_py: geometry collision box size=0.3 0.025 0.5; visual box size=0.3 0.025 0.5
Joints:
- joint edge_joint_nx: origin xyz=-0.225 0 0 -> xyz=-0.1455 0 0
- joint edge_joint_ny: origin xyz=0 -0.225 0 -> xyz=0 -0.1455 0
- joint edge_joint_px: origin xyz=0.225 0 0 -> xyz=0.1455 0 0
- joint edge_joint_py: origin xyz=0 0.225 0 -> xyz=0 0.1455 0

File: robo_manip_baselines/envs/assets/tacto/objects/box/white_box.urdf (robot description, URDF)
Before this commit: robot white_box.urdf, 5 links, 4 joints
Links:
- link bottom: geometry collision box size=0.3 0.3 0.1; visual box size=0.3 0.3 0.1
- link edge_nx: geometry collision box size=0.025 0.3 0.5; visual box size=0.025 0.3 0.5
- link edge_ny: geometry collision box size=0.3 0.025 0.5; visual box size=0.3 0.025 0.5
- link edge_px: geometry collision box size=0.025 0.3 0.5; visual box size=0.025 0.3 0.5
- link edge_py: geometry collision box size=0.3 0.025 0.5; visual box size=0.3 0.025 0.5
Joints:
- joint edge_joint_nx: origin xyz=-0.225 0 0 -> xyz=-0.1455 0 0
- joint edge_joint_ny: origin xyz=0 -0.225 0 -> xyz=0 -0.1455 0
- joint edge_joint_px: origin xyz=0.225 0 0 -> xyz=0.1455 0 0
- joint edge_joint_py: origin xyz=0 0.225 0 -> xyz=0 0.1455 0
